File: KB1/KB1.kicad_pcb (KiCad board)
At the start: 2 copper layers, 24 parts, among them SW1 SW_Push, U1 ATmega32U4-AU, Y1 16MHz

Commit message: pcb routing addition
Parts:
- moved C7 8.66 mm to (346.2, 236.2), turned to 270 degrees
- moved C3 5.61 mm to (366.6, 217.9)
- moved C2 5.61 mm to (357.9, 217.9)
- moved Y1 5.61 mm to (362.4, 217.9)
- moved R2 5.59 mm to (343.6, 217.6)
- moved R1 5.37 mm to (340.1, 217.6)
- moved R3 5.00 mm to (346.3, 222.4)
- moved C5 4.55 mm to (348.6, 222.4)
- moved C6 1.80 mm to (344.3, 228.4), turned to 180 degrees
- turned F1 to 90 degrees
Connections:
- U1 pad 27: Net-(U1-Pad27) -> ROW0
- U1 pad 28: Net-(U1-Pad28) -> COL1
- U1 pad 29: Net-(U1-Pad29) -> COL0
- U1 pad 30: Net-(U1-Pad30) -> ROW1
Routing:
- net GND: track 0.00 -> 143.7 mm, vias 0 -> 2
- net +5V: track 0.00 -> 100.3 mm, vias 0 -> 2
- net COL1: track 0.00 -> 61.1 mm
- net ROW0: track 0.00 -> 57.2 mm
- net ROW1: track 0.00 -> 54.8 mm
- net Net-(R3-Pad2): track 0.00 -> 41.1 mm, vias 0 -> 2
- net COL0: track 0.00 -> 40.5 mm
- net Net-(C2-Pad1): track 0.00 -> 30.7 mm
- net Net-(R1-Pad1): track 0.00 -> 22.7 mm
- net Net-(R2-Pad1): track 0.00 -> 21.1 mm
- net VCC: track 0.00 -> 15.2 mm
- net Net-(C3-Pad1): track 0.00 -> 13.7 mm
- net Net-(C6-Pad1): track 0.00 -> 6.75 mm
- net Net-(D2-Pad2): track 0.00 -> 6.62 mm
- net Net-(D4-Pad2): track 0.00 -> 6.62 mm
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